File: SWR bridge.kicad_pcb (KiCad board)
At the start: 2 copper layers, 107.5 x 46 mm, 20 parts, among them J1 Conn_Coaxial, J10 Conn_01x01_Male, J2 Conn_01x01_Female, J3 Conn_Coaxial, J4 Conn_01x01_Female, J5 Conn_01x01_Female, J6 Conn_01x01_Female, J7 Conn_01x01_Male, J8 Conn_01x01_Male, J9 Conn_01x01_Male

Commit message: Add files via upload
Parts:
- added R3: 1,5K, Resistor_THT:R_Axial_DIN0204_L3.6mm_D1.6mm_P5.08mm_Horizontal, F.Cu at (116.0, 42.5)
- added R4: 1K, Resistor_THT:R_Axial_DIN0204_L3.6mm_D1.6mm_P5.08mm_Horizontal, F.Cu at (120.0, 36.0)
- added R5: 1,5K, Resistor_THT:R_Axial_DIN0204_L3.6mm_D1.6mm_P5.08mm_Horizontal, F.Cu at (116.0, 71.9)
- added R6: 1K, Resistor_THT:R_Axial_DIN0204_L3.6mm_D1.6mm_P5.08mm_Horizontal, F.Cu at (119.4, 78.5)
- added REF**: MountingHole_2.2mm_M2_DIN965_Pad, MountingHole:MountingHole_2.2mm_M2_DIN965_Pad, F.Cu at (147.5, 76.0)
- added REF**: MountingHole_2.2mm_M2_DIN965_Pad, MountingHole:MountingHole_2.2mm_M2_DIN965_Pad, F.Cu at (136.5, 76.0)
- added REF**: MountingHole_2.2mm_M2_DIN965_Pad, MountingHole:MountingHole_2.2mm_M2_DIN965_Pad, F.Cu at (147.0, 38.5)
- added REF**: MountingHole_2.2mm_M2_DIN965_Pad, MountingHole:MountingHole_2.2mm_M2_DIN965_Pad, F.Cu at (136.5, 38.5)
- added REF**: MountingHole_2.2mm_M2_DIN965_Pad, MountingHole:MountingHole_2.2mm_M2_DIN965_Pad, F.Cu at (129.5, 68.0)
- added REF**: MountingHole_2.2mm_M2_DIN965_Pad, MountingHole:MountingHole_2.2mm_M2_DIN965_Pad, F.Cu at (120.0, 68.0)
- added REF**: MountingHole_2.2mm_M2_DIN965_Pad, MountingHole:MountingHole_2.2mm_M2_DIN965_Pad, F.Cu at (129.5, 46.5)
- added REF**: MountingHole_2.2mm_M2_DIN965_Pad, MountingHole:MountingHole_2.2mm_M2_DIN965_Pad, F.Cu at (120.0, 46.5)
- D1: value 1N4148 -> 1N5711
- moved C3 3.16 mm to (120.0, 40.5)
- moved C4 2.00 mm to (119.5, 74.0)
- moved R2 0.50 mm to (87.5, 37.5)
- moved J2 0.42 mm to (111.5, 37.0)
Connections:
- J2 pad 1: /REF -> /vREF
- J6 pad 1: /FORWARD -> /VFOR
Routing:
- net /T1: track 59.5 -> 43.7 mm, vias 0 -> 1
- net /vREF: track 0.00 -> 10.2 mm
- net /VFOR: track 0.00 -> 8.04 mm
- net /FORWARD: track 12.8 -> 14.8 mm
- net /REF: track 13.8 -> 15.8 mm
- net /T-center: track 57.5 -> 56.5 mm

Commit message: Add files via upload
updated files
Parts:
- removed REF** (x8): MountingHole_2.2mm_M2_DIN965_Pad, MountingHole:MountingHole_2.2mm_M2_DIN965_Pad
- added C6: 100nF, Capacitor_THT:C_Disc_D7.5mm_W5.0mm_P7.50mm, F.Cu at (72.5, 37.5)
- added D3: 1N5711, Diode_THT:D_DO-35_SOD27_P7.62mm_Horizontal, F.Cu at (66.0, 48.5)
- added J11: Conn_01x01_Female, Connector_PinHeader_1.00mm:PinHeader_1x01_P1.00mm_Vertical, F.Cu at (61.0, 36.5)
- added J12: Conn_01x01_Male, MountingHole:MountingHole_2.2mm_M2_DIN965_Pad, F.Cu at (119.5, 67.0)
- added J13: Conn_01x01_Male, MountingHole:MountingHole_2.2mm_M2_DIN965_Pad, F.Cu at (136.0, 37.5)
- added J14: Conn_01x01_Male, MountingHole:MountingHole_2.2mm_M2_DIN965_Pad, F.Cu at (130.5, 47.0)
- added J15: Conn_01x01_Male, MountingHole:MountingHole_2.2mm_M2_DIN965_Pad, F.Cu at (148.0, 37.5)
- added J16: Conn_01x01_Male, MountingHole:MountingHole_2.2mm_M2_DIN965_Pad, F.Cu at (130.5, 67.0)
- added J17: Conn_01x01_Male, MountingHole:MountingHole_2.2mm_M2_DIN965_Pad, F.Cu at (136.0, 76.5)
- added J18: Conn_01x01_Male, MountingHole:MountingHole_2.2mm_M2_DIN965_Pad, F.Cu at (120.0, 47.0)
- added J19: Conn_01x01_Male, MountingHole:MountingHole_2.2mm_M2_DIN965_Pad, F.Cu at (148.0, 76.5)
- added L1: 100uH, Resistor_THT:R_Axial_DIN0204_L3.6mm_D1.6mm_P7.62mm_Horizontal, F.Cu at (66.0, 44.1)
- added L3: 100uH, Resistor_THT:R_Axial_DIN0204_L3.6mm_D1.6mm_P7.62mm_Horizontal, F.Cu at (114.0, 43.6)
- added L4: 100uH, Resistor_THT:R_Axial_DIN0204_L3.6mm_D1.6mm_P7.62mm_Horizontal, F.Cu at (114.0, 77.6)
- moved J6 1.00 mm to (111.0, 77.0)
- moved J2 0.71 mm to (111.0, 36.5)
- moved R5 0.65 mm to (116.5, 71.5)
- moved C4 0.50 mm to (119.5, 73.5)
- moved R3 0.50 mm to (116.5, 42.5)
- moved R6 0.50 mm to (119.4, 78.0)
Connections:
- J2 pad 1: /vREF -> Net-(J2-Pad1)
- J6 pad 1: /VFOR -> Net-(J6-Pad1)
Routing:
- net Net-(C6-Pad1): track 0.00 -> 13.7 mm
- net Net-(J11-Pad1): track 0.00 -> 5.00 mm
- net /VFOR: track 8.04 -> 11.9 mm
- net Net-(J2-Pad1): track 0.00 -> 3.21 mm
- net Net-(J6-Pad1): track 0.00 -> 3.05 mm
- net /vREF: track 10.2 -> 11.2 mm
Other:
- board text added: "FV"
- board text added: "KF"
- board text added: "RV"
- board text added: "TO ANT"
- board text removed: "ANT"
- board text removed: "FORWARD"
- board text removed: "REVERSE"

Commit message: Add files via upload
update
Parts:
- removed C6: 100nF, Capacitor_THT:C_Disc_D7.5mm_W5.0mm_P7.50mm
- removed D3: 1N5711, Diode_THT:D_DO-35_SOD27_P7.62mm_Horizontal
- removed J11: Conn_01x01_Female, Connector_PinHeader_1.00mm:PinHeader_1x01_P1.00mm_Vertical
- removed L1: 100uH, Resistor_THT:R_Axial_DIN0204_L3.6mm_D1.6mm_P7.62mm_Horizontal
Routing:
- net Net-(C6-Pad1): track 13.7 -> 0.00 mm
- net Net-(J11-Pad1): track 5.00 -> 0.00 mm
Other:
- board text added: "160m-6m"
